File: pcb.kicad_pcb (KiCad board)
At the start: 4 copper layers, 40 x 44 mm, 45 parts, among them J1 USB_C_Receptacle_USB2.0, J2 Conn_ARM_JTAG_SWD_10, J3 Conn_02x25_Counter_Clockwise, SW1 SW_Push, SW2 SW_Push, U1 25CSM04, U2 EFM32GG11B8xx-QFN64, U3 74LVC1G17, U4 MIC2003, Y1 32.768KHz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

Commit message: production fixes
Routing:
- net GND: track 44.8 -> 46.8 mm, vias 44 -> 46
- net Net-(J3-Pad47): vias 6 -> 5
Other:
- board text added: "JLCJLCJLCJLC"
